Commit message: Added goalie from white team Not sure about the way I did it.  Tried to have a ghost joint so I could include both translation and rotation, but did not work.  Instead have rod translate and players rotate around rod (don't love that but oh well).  Will try to think of another way to make it work.

File: Code/simulation/CollisionTable.urdf (robot description, URDF)
Before this commit: robot collision_table, 1 links, 0 joints
Links:
- added link goaliePlayer11; collision mesh filename=PlayerCollider.obj scale=.001 .001 .001; visual mesh filename=PlayerVisual.obj scale=.001 .001 .001
- added link goaliePlayer12; collision mesh filename=PlayerCollider.obj scale=.001 .001 .001; visual mesh filename=PlayerVisual.obj scale=.001 .001 .001
- added link goaliePlayer13; collision mesh filename=PlayerCollider.obj scale=.001 .001 .001; visual mesh filename=PlayerVisual.obj scale=.001 .001 .001
- added link goalieRod1; collision cylinder length=1 radius=.0078613; visual mesh filename=GoalieRod.obj scale=.001 .001 .001
Joints:
- added joint GP11: type continuous, parent goalieRod1, child goaliePlayer11, origin xyz=0 0.250825 0 rpy=0 0 1.5707963, axis 0 1 0
- added joint GP12: type continuous, parent goalieRod1, child goaliePlayer12, origin xyz=0 0.4572 0 rpy=0 0 1.5707963, axis 0 1 0
- added joint GP13: type continuous, parent goalieRod1, child goaliePlayer13, origin xyz=0 0.663575 0 rpy=0 0 1.5707963, axis 0 1 0
- added joint goaliePrismatic1: type prismatic, parent baseLink, child goalieRod1, origin xyz=0.508 -0.366395 0.098425 rpy=0 0 0, axis 0 -1 0, limit lower=0 upper=.18161

Commit message: urdf updates, still trying to track down ball speed during striker start

File: Code/simulation/CollisionTable.urdf (robot description, URDF)
Before this commit: robot collision_table, 5 links, 4 joints
Links:
- added link defenseBlock1, mass 1; collision box size=.0625 .03125 .125; visual box size=.0625 .03125 .125
- added link defenseBlock2, mass 1; collision box size=.0625 .03125 .125; visual box size=.0625 .03125 .125
- added link defensePlayer11, mass 1; collision mesh filename=PlayerCollider.obj scale=.001 .001 .001; visual mesh filename=PlayerVisual.obj scale=.001 .001 .001
- added link defensePlayer12, mass 1; collision mesh filename=PlayerCollider.obj scale=.001 .001 .001; visual mesh filename=PlayerVisual.obj scale=.001 .001 .001
- added link defensePlayer21, mass 1; collision mesh filename=PlayerCollider.obj scale=.001 .001 .001; visual mesh filename=PlayerVisual.obj scale=.001 .001 .001
- added link defensePlayer22, mass 1; collision mesh filename=PlayerCollider.obj scale=.001 .001 .001; visual mesh filename=PlayerVisual.obj scale=.001 .001 .001
- added link defenseRod1, mass 1; collision cylinder length=1.228725 radius=0.0078613; visual cylinder length=1.228725 radius=0.0078613
- added link defenseRod2, mass 1; collision cylinder length=1.228725 radius=0.0078613; visual cylinder length=1.228725 radius=0.0078613
- added link goalieBlock1, mass 1; collision box size=.0625 .03125 .125; visual box size=.0625 .03125 .125
- added link goalieBlock2, mass 1; collision box size=.0625 .03125 .125; visual box size=.0625 .03125 .125
- added link goaliePlayer21, mass 1; collision mesh filename=PlayerCollider.obj scale=.001 .001 .001; visual mesh filename=PlayerVisual.obj scale=.001 .001 .001
- added link goaliePlayer22, mass 1; collision mesh filename=PlayerCollider.obj scale=.001 .001 .001; visual mesh filename=PlayerVisual.obj scale=.001 .001 .001
- added link goaliePlayer23, mass 1; collision mesh filename=PlayerCollider.obj scale=.001 .001 .001; visual mesh filename=PlayerVisual.obj scale=.001 .001 .001
- added link goalieRod2, mass 1; collision cylinder length=1.0541 radius=0.0078613; visual cylinder length=1.0541 radius=0.0078613
- added link midfieldBlock1, mass 1; collision box size=.0625 .03125 .125; visual box size=.0625 .03125 .125
- added link midfieldBlock2, mass 1; collision box size=.0625 .03125 .125; visual box size=.0625 .03125 .125
- added link midfieldPlayer11, mass 1; collision mesh filename=PlayerCollider.obj scale=.001 .001 .001; visual mesh filename=PlayerVisual.obj scale=.001 .001 .001
- added link midfieldPlayer12, mass 1; collision mesh filename=PlayerCollider.obj scale=.001 .001 .001; visual mesh filename=PlayerVisual.obj scale=.001 .001 .001
- added link midfieldPlayer13, mass 1; collision mesh filename=PlayerCollider.obj scale=.001 .001 .001; visual mesh filename=PlayerVisual.obj scale=.001 .001 .001
- added link midfieldPlayer14, mass 1; collision mesh filename=PlayerCollider.obj scale=.001 .001 .001; visual mesh filename=PlayerVisual.obj scale=.001 .001 .001
- added link midfieldPlayer15, mass 1; collision mesh filename=PlayerCollider.obj scale=.001 .001 .001; visual mesh filename=PlayerVisual.obj scale=.001 .001 .001
- added link midfieldPlayer21, mass 1; collision mesh filename=PlayerCollider.obj scale=.001 .001 .001; visual mesh filename=PlayerVisual.obj scale=.001 .001 .001
- added link midfieldPlayer22, mass 1; collision mesh filename=PlayerCollider.obj scale=.001 .001 .001; visual mesh filename=PlayerVisual.obj scale=.001 .001 .001
- added link midfieldPlayer23, mass 1; collision mesh filename=PlayerCollider.obj scale=.001 .001 .001; visual mesh filename=PlayerVisual.obj scale=.001 .001 .001
- added link midfieldPlayer24, mass 1; collision mesh filename=PlayerCollider.obj scale=.001 .001 .001; visual mesh filename=PlayerVisual.obj scale=.001 .001 .001
- added link midfieldPlayer25, mass 1; collision mesh filename=PlayerCollider.obj scale=.001 .001 .001; visual mesh filename=PlayerVisual.obj scale=.001 .001 .001
- added link midfieldRod1, mass 1; collision cylinder length=0.987425 radius=0.0078613; visual cylinder length=0.987425 radius=0.0078613
- added link midfieldRod2, mass 1; collision cylinder length=0.987425 radius=0.0078613; visual cylinder length=0.987425 radius=0.0078613
- added link strikerBlock1, mass 1; collision box size=.0625 .03125 .125; visual box size=.0625 .03125 .125
- added link strikerBlock2, mass 1; collision box size=.0625 .03125 .125; visual box size=.0625 .03125 .125
- added link strikerPlayer11, mass 1; collision mesh filename=PlayerCollider.obj scale=.001 .001 .001; visual mesh filename=PlayerVisual.obj scale=.001 .001 .001
- added link strikerPlayer12, mass 1; collision mesh filename=PlayerCollider.obj scale=.001 .001 .001; visual mesh filename=PlayerVisual.obj scale=.001 .001 .001
- added link strikerPlayer13, mass 1; collision mesh filename=PlayerCollider.obj scale=.001 .001 .001; visual mesh filename=PlayerVisual.obj scale=.001 .001 .001
- added link strikerPlayer21, mass 1; collision mesh filename=PlayerCollider.obj scale=.001 .001 .001; visual mesh filename=PlayerVisual.obj scale=.001 .001 .001
- added link strikerPlayer22, mass 1; collision mesh filename=PlayerCollider.obj scale=.001 .001 .001; visual mesh filename=PlayerVisual.obj scale=.001 .001 .001
- added link strikerPlayer23, mass 1; collision mesh filename=PlayerCollider.obj scale=.001 .001 .001; visual mesh filename=PlayerVisual.obj scale=.001 .001 .001
- added link strikerRod1, mass 1; collision cylinder length=1.101725 radius=0.0078613; visual cylinder length=1.101725 radius=0.0078613
- added link strikerRod2, mass 1; collision cylinder length=1.101725 radius=0.0078613; visual cylinder length=1.101725 radius=0.0078613
- link goaliePlayer11: mass None -> 1
- link goaliePlayer12: mass None -> 1
- link goaliePlayer13: mass None -> 1
- link goalieRod1: mass None -> 1; geometry collision cylinder length=1.0541 radius=0.0078613; visual cylinder length=1.0541 radius=0.0078613
Joints:
- added joint DP11: type fixed, parent defenseRod1, child defensePlayer11, origin xyz=0 0.41021 0 rpy=0 0 1.5707963267948966
- added joint DP12: type fixed, parent defenseRod1, child defensePlayer12, origin xyz=0 0.65151 0 rpy=0 0 1.5707963267948966
- added joint DP21: type fixed, parent defenseRod2, child defensePlayer21, origin xyz=0 0.41021 0 rpy=0 0 1.5707963267948966
- added joint DP22: type fixed, parent defenseRod2, child defensePlayer22, origin xyz=0 0.65151 0 rpy=0 0 1.5707963267948966
- added joint GP21: type fixed, parent goalieRod2, child goaliePlayer21, origin xyz=0 0.235585 0 rpy=0 0 1.5707963267948966
- added joint GP22: type fixed, parent goalieRod2, child goaliePlayer22, origin xyz=0 0.44196 0 rpy=0 0 1.5707963267948966
- added joint GP23: type fixed, parent goalieRod2, child goaliePlayer23, origin xyz=0 0.648335 0 rpy=0 0 1.5707963267948966
- added joint MP11: type fixed, parent midfieldRod1, child midfieldPlayer11, origin xyz=0 0.16891 0 rpy=0 0 1.5707963267948966
- added joint MP12: type fixed, parent midfieldRod1, child midfieldPlayer12, origin xyz=0 0.28956 0 rpy=0 0 1.5707963267948966
- added joint MP13: type fixed, parent midfieldRod1, child midfieldPlayer13, origin xyz=0 0.4191 0 rpy=0 0 1.5707963267948966
- added joint MP14: type fixed, parent midfieldRod1, child midfieldPlayer14, origin xyz=0 0.53086 0 rpy=0 0 1.5707963267948966
- added joint MP15: type fixed, parent midfieldRod1, child midfieldPlayer15, origin xyz=0 0.65151 0 rpy=0 0 1.5707963267948966
- added joint MP21: type fixed, parent midfieldRod2, child midfieldPlayer21, origin xyz=0 0.16891 0 rpy=0 0 1.5707963267948966
- added joint MP22: type fixed, parent midfieldRod2, child midfieldPlayer22, origin xyz=0 0.28956 0 rpy=0 0 1.5707963267948966
- added joint MP23: type fixed, parent midfieldRod2, child midfieldPlayer23, origin xyz=0 0.4191 0 rpy=0 0 1.5707963267948966
- added joint MP24: type fixed, parent midfieldRod2, child midfieldPlayer24, origin xyz=0 0.53086 0 rpy=0 0 1.5707963267948966
- added joint MP25: type fixed, parent midfieldRod2, child midfieldPlayer25, origin xyz=0 0.65151 0 rpy=0 0 1.5707963267948966
- added joint SP11: type fixed, parent strikerRod1, child strikerPlayer11, origin xyz=0 0.28321 0 rpy=0 0 1.5707963267948966
- added joint SP12: type fixed, parent strikerRod1, child strikerPlayer12, origin xyz=0 0.46736 0 rpy=0 0 1.5707963267948966
- added joint SP13: type fixed, parent strikerRod1, child strikerPlayer13, origin xyz=0 0.65151 0 rpy=0 0 1.5707963267948966
- added joint SP21: type fixed, parent strikerRod2, child strikerPlayer21, origin xyz=0 0.28321 0 rpy=0 0 1.5707963267948966
- added joint SP22: type fixed, parent strikerRod2, child strikerPlayer22, origin xyz=0 0.46736 0 rpy=0 0 1.5707963267948966
- added joint SP23: type fixed, parent strikerRod2, child strikerPlayer23, origin xyz=0 0.65151 0 rpy=0 0 1.5707963267948966
- added joint defensePrismatic1: type prismatic, parent baseLink, child defenseBlock1, origin xyz=0.36195 0.859155 0 rpy=0 0 3.14159265, axis 0 1 0, limit lower=0 upper=.35306
- added joint defensePrismatic2: type prismatic, parent baseLink, child defenseBlock2, origin xyz=-0.36195 -0.859155 0 rpy=0 0 0, axis 0 1 0, limit lower=0 upper=.35306
- added joint defenseRotation1: type continuous, parent defenseBlock1, child defenseRod1, origin xyz=0 1.228725 0.098425 rpy=0 0 3.14152965, axis 0 1 0
- added joint defenseRotation2: type continuous, parent defenseBlock2, child defenseRod2, origin xyz=0 1.228725 0.098425 rpy=0 0 3.14159265, axis 0 1 0
- added joint goaliePrismatic2: type prismatic, parent baseLink, child goalieBlock2, origin xyz=-0.508 -0.687705 0 rpy=0 0 0, axis 0 1 0, limit lower=0 upper=.18161
- added joint goalieRotation1: type continuous, parent goalieBlock1, child goalieRod1, origin xyz=0 1.0541 0.098425 rpy=0 0 3.14159265, axis 0 1 0
- added joint goalieRotation2: type continuous, parent goalieBlock2, child goalieRod2, origin xyz=0 1.0541 0.098425 rpy=0 0 3.14159265, axis 0 1 0
- added joint midfieldPrismatic1: type prismatic, parent baseLink, child midfieldBlock1, origin xyz=0.066675 0.617855 0 rpy=0 0 3.14159265, axis 0 1 0, limit lower=0 upper=.11176
- added joint midfieldPrismatic2: type prismatic, parent baseLink, child midfieldBlock2, origin xyz=-0.066675 -0.617855 0 rpy=0 0 0, axis 0 1 0, limit lower=0 upper=.11176
- added joint midfieldRotation1: type continuous, parent midfieldBlock1, child midfieldRod1, origin xyz=0 0.987425 0.098425 rpy=0 0 3.14159265, axis 0 1 0
- added joint midfieldRotation2: type continuous, parent midfieldBlock2, child midfieldRod2, origin xyz=0 0.987425 0.098425 rpy=0 0 3.14159265, axis 0 1 0
- added joint strikerPrismatic1: type prismatic, parent baseLink, child strikerBlock1, origin xyz=-0.2159 0.732155 0 rpy=0 0 3.14159265, axis 0 1 0, limit lower=0 upper=.22606
- added joint strikerPrismatic2: type prismatic, parent baseLink, child strikerBlock2, origin xyz=0.2159 -0.732155 0 rpy=0 0 0, axis 0 1 0, limit lower=0 upper=.22606
- added joint strikerRotation1: type continuous, parent strikerBlock1, child strikerRod1, origin xyz=0 1.101725 0.098425 rpy=0 0 3.14159265, axis 0 1 0
- added joint strikerRotation2: type continuous, parent strikerBlock2, child strikerRod2, origin xyz=0 1.101725 0.098425 rpy=0 0 3.14159265, axis 0 1 0
- joint GP11: axis 0 1 0 -> (none); origin xyz=0 0.250825 0 rpy=0 0 1.5707963 -> xyz=0 0.235585 0 rpy=0 0 1.5707963267948966; type continuous -> fixed
- joint GP12: axis 0 1 0 -> (none); origin xyz=0 0.4572 0 rpy=0 0 1.5707963 -> xyz=0 0.44196 0 rpy=0 0 1.5707963267948966; type continuous -> fixed
- joint GP13: axis 0 1 0 -> (none); origin xyz=0 0.663575 0 rpy=0 0 1.5707963 -> xyz=0 0.648335 0 rpy=0 0 1.5707963267948966; type continuous -> fixed
- joint goaliePrismatic1: axis 0 -1 0 -> 0 1 0; child goalieRod1 -> goalieBlock1; origin xyz=0.508 -0.366395 0.098425 rpy=0 0 0 -> xyz=0.508 0.687705 0 rpy=0 0 3.14159265

File: Code/simulation/TableTest.urdf (robot description, URDF)
Before this commit: robot collision_table, 43 links, 42 joints
Links:
- link defenseRod1: geometry collision cylinder length=${defenseLength} radius=${rodRadius}; visual cylinder length=${defenseLength} radius=${rodRadius}
- link defenseRod2: geometry collision cylinder length=${defenseLength} radius=${rodRadius}; visual cylinder length=${defenseLength} radius=${rodRadius}
- link goalieRod1: geometry collision cylinder length=${goalieLength} radius=${rodRadius}; visual cylinder length=${goalieLength} radius=${rodRadius}
- link goalieRod2: geometry collision cylinder length=${goalieLength} radius=${rodRadius}; visual cylinder length=${goalieLength} radius=${rodRadius}
- link midfieldRod1: geometry collision cylinder length=${midfieldLength} radius=${rodRadius}; visual cylinder length=${midfieldLength} radius=${rodRadius}
- link midfieldRod2: geometry collision cylinder length=${midfieldLength} radius=${rodRadius}; visual cylinder length=${midfieldLength} radius=${rodRadius}
- link strikerRod1: geometry collision cylinder length=${strikerLength} radius=${rodRadius}; visual cylinder length=${strikerLength} radius=${rodRadius}
- link strikerRod2: geometry collision cylinder length=${strikerLength} radius=${rodRadius}; visual cylinder length=${strikerLength} radius=${rodRadius}
Joints:
- joint DP11: origin xyz=0 0.41021 0 rpy=0 0 1.5707963 -> xyz=0 0.41021 0 rpy=0 0 ${pi/2}
- joint DP12: origin xyz=0 0.65151 0 rpy=0 0 1.5707963 -> xyz=0 0.65151 0 rpy=0 0 ${pi/2}
- joint DP21: origin xyz=0 0.41021 0 rpy=0 0 1.5707963 -> xyz=0 0.41021 0 rpy=0 0 ${pi/2}
- joint DP22: origin xyz=0 0.65151 0 rpy=0 0 1.5707963 -> xyz=0 0.65151 0 rpy=0 0 ${pi/2}
- joint GP11: origin xyz=0 0.235585 0 rpy=0 0 1.5707963 -> xyz=0 0.235585 0 rpy=0 0 ${pi/2}
- joint GP12: origin xyz=0 0.44196 0 rpy=0 0 1.5707963 -> xyz=0 0.44196 0 rpy=0 0 ${pi/2}
- joint GP13: origin xyz=0 0.648335 0 rpy=0 0 1.5707963 -> xyz=0 0.648335 0 rpy=0 0 ${pi/2}
- joint GP21: origin xyz=0 0.235585 0 rpy=0 0 1.5707963 -> xyz=0 0.235585 0 rpy=0 0 ${pi/2}
- joint GP22: origin xyz=0 0.44196 0 rpy=0 0 1.5707963 -> xyz=0 0.44196 0 rpy=0 0 ${pi/2}
- joint GP23: origin xyz=0 0.648335 0 rpy=0 0 1.5707963 -> xyz=0 0.648335 0 rpy=0 0 ${pi/2}
- joint MP11: origin xyz=0 0.16891 0 rpy=0 0 1.5707963 -> xyz=0 0.16891 0 rpy=0 0 ${pi/2}
- joint MP12: origin xyz=0 0.28956 0 rpy=0 0 1.5707963 -> xyz=0 0.28956 0 rpy=0 0 ${pi/2}
- joint MP13: origin xyz=0 0.4191 0 rpy=0 0 1.5707963 -> xyz=0 0.4191 0 rpy=0 0 ${pi/2}
- joint MP14: origin xyz=0 0.53086 0 rpy=0 0 1.5707963 -> xyz=0 0.53086 0 rpy=0 0 ${pi/2}
- joint MP15: origin xyz=0 0.65151 0 rpy=0 0 1.5707963 -> xyz=0 0.65151 0 rpy=0 0 ${pi/2}
- joint MP21: origin xyz=0 0.16891 0 rpy=0 0 1.5707963 -> xyz=0 0.16891 0 rpy=0 0 ${pi/2}
- joint MP22: origin xyz=0 0.28956 0 rpy=0 0 1.5707963 -> xyz=0 0.28956 0 rpy=0 0 ${pi/2}
- joint MP23: origin xyz=0 0.4191 0 rpy=0 0 1.5707963 -> xyz=0 0.4191 0 rpy=0 0 ${pi/2}
- joint MP24: origin xyz=0 0.53086 0 rpy=0 0 1.5707963 -> xyz=0 0.53086 0 rpy=0 0 ${pi/2}
- joint MP25: origin xyz=0 0.65151 0 rpy=0 0 1.5707963 -> xyz=0 0.65151 0 rpy=0 0 ${pi/2}
- joint SP11: origin xyz=0 0.28321 0 rpy=0 0 1.5707963 -> xyz=0 0.28321 0 rpy=0 0 ${pi/2}
- joint SP12: origin xyz=0 0.46736 0 rpy=0 0 1.5707963 -> xyz=0 0.46736 0 rpy=0 0 ${pi/2}
- joint SP13: origin xyz=0 0.65151 0 rpy=0 0 1.5707963 -> xyz=0 0.65151 0 rpy=0 0 ${pi/2}
- joint SP21: origin xyz=0 0.28321 0 rpy=0 0 1.5707963 -> xyz=0 0.28321 0 rpy=0 0 ${pi/2}
- joint SP22: origin xyz=0 0.46736 0 rpy=0 0 1.5707963 -> xyz=0 0.46736 0 rpy=0 0 ${pi/2}
- joint SP23: origin xyz=0 0.65151 0 rpy=0 0 1.5707963 -> xyz=0 0.65151 0 rpy=0 0 ${pi/2}
- joint midfieldRotation1: origin xyz=0 0.987425 0.098425 rpy=0 0 3.14159265 -> xyz=0 ${midfieldLength} 0.098425 rpy=0 0 3.14159265
- joint midfieldRotation2: origin xyz=0 0.987425 0.098425 rpy=0 0 3.14159265 -> xyz=0 ${midfieldLength} 0.098425 rpy=0 0 3.14159265
- joint strikerRotation1: origin xyz=0 1.101725 0.098425 rpy=0 0 3.14159265 -> xyz=0 ${strikerLength} 0.098425 rpy=0 0 3.14159265
- joint strikerRotation2: origin xyz=0 1.101725 0.098425 rpy=0 0 3.14159265 -> xyz=0 ${strikerLength} 0.098425 rpy=0 0 3.14159265
